File: board/milki.kicad_pcb (KiCad board)
At the start: 2 copper layers, 228.6 x 81 mm, 81 parts

Commit message: i've switched up
Parts:
- A1: value RaspberryPi_Pico -> Arduino_Nano_Every; footprint Module:RaspberryPi_Pico_Common_Unspecified -> Module:Arduino_Nano
- MX1, MX10, MX11, MX12, MX13, MX14, MX15, MX16, MX17, MX18, MX19, MX2, MX20, MX21, MX22, MX23, MX24, MX25, MX26, MX27, MX28, MX29, MX3, MX30, MX31, MX32, MX33, MX34, MX35, MX36, MX37, MX38, MX39, MX4, MX40, MX5, MX6, MX7, MX8, MX9: footprint PCM_marbastlib-xp-alps:SW_Alps_MX_1u -> MX_Solderable:Low Profile GC plus MX
- moved D10 281.2 mm to (24.4, 176.1), turned to 0 degrees
- moved D9 262.9 mm to (24.4, 172.6), turned to 0 degrees
- moved D20 261.1 mm to (35.1, 172.6), turned to 0 degrees
- moved D8 244.6 mm to (24.4, 169.0), turned to 0 degrees
- moved D19 242.4 mm to (35.1, 169.0), turned to 0 degrees
- moved D30 242.2 mm to (45.9, 169.0), turned to 0 degrees
- moved D7 226.6 mm to (24.4, 165.5), turned to 0 degrees
- moved D40 224.5 mm to (56.7, 165.5), turned to 0 degrees
- moved D18 223.8 mm to (35.1, 165.5), turned to 0 degrees
- moved D29 223.2 mm to (45.9, 165.5), turned to 0 degrees
- moved D6 208.9 mm to (24.4, 161.9), turned to 0 degrees
- moved D17 205.4 mm to (35.1, 161.9), turned to 0 degrees
- moved D39 205.3 mm to (56.7, 161.9), turned to 0 degrees
- moved D28 204.3 mm to (45.9, 161.9), turned to 0 degrees
- moved D16 187.2 mm to (35.1, 158.4), turned to 0 degrees
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Connections:
- A1 pad 10: /Col 1 -> unconnected-(A1-D7-Pad10)
- A1 pad 11: /Col 2 -> unconnected-(A1-D8-Pad11)
- A1 pad 12: /Col 3 -> unconnected-(A1-D9-Pad12)
- A1 pad 13: Net-(A1-GND-Pad13) -> unconnected-(A1-D10-Pad13)
- A1 pad 14: /Col 4 -> unconnected-(A1-MOSI-Pad14)
- A1 pad 15: /Col 5 -> unconnected-(A1-MISO-Pad15)
- A1 pad 16: /Col 6 -> unconnected-(A1-SCK-Pad16)
- A1 pad 17: /Col 7 -> unconnected-(A1-3V3-Pad17)
- A1 pad 18: Net-(A1-GND-Pad13) -> unconnected-(A1-AREF-Pad18)
- A1 pad 19: /Col 8 -> unconnected-(A1-A0-Pad19)
- A1 pad 20: /Col 9 -> unconnected-(A1-A1-Pad20)
- A1 pad 21: /Row 0 -> unconnected-(A1-A2-Pad21)
- A1 pad 22: /Row 1 -> unconnected-(A1-A3-Pad22)
- A1 pad 23: Net-(A1-GND-Pad13) -> unconnected-(A1-SDA/A4-Pad23)
- A1 pad 24: /Row 2 -> unconnected-(A1-SCL/A5-Pad24)
- A1 pad 25: /Row 3 -> unconnected-(A1-A6-Pad25)
- A1 pad 28: Net-(A1-GND-Pad13) -> unconnected-(A1-~{RESET}-Pad28)
- A1 pad 29: unconnected-(A1-GPIO22-Pad29) -> Net-(A1-GND-Pad29)
- A1 pad 3: Net-(A1-GND-Pad13) -> unconnected-(A1-~{RESET}-Pad3)
- A1 pad 4: unconnected-(A1-GPIO2-Pad4) -> Net-(A1-GND-Pad29)
- A1 pad 8: Net-(A1-GND-Pad13) -> unconnected-(A1-D5-Pad8)
- A1 pad 9: /Col 0 -> unconnected-(A1-D6-Pad9)
- D10 pad 1: /Row 0 -> /Row 1
- D11 pad 1: /Row 1 -> /Row 2
- D12 pad 1: /Row 1 -> /Row 2
- D13 pad 1: /Row 1 -> /Row 2
- D14 pad 1: /Row 1 -> /Row 2
- D15 pad 1: /Row 1 -> /Row 2
- D16 pad 1: /Row 1 -> /Row 3
- D17 pad 1: /Row 1 -> /Row 3
- D18 pad 1: /Row 1 -> /Row 3
- D19 pad 1: /Row 1 -> /Row 3
- D20 pad 1: /Row 1 -> /Row 3
- D21 pad 1: /Row 2 -> /Row 0
- D22 pad 1: /Row 2 -> /Row 1
- D24 pad 1: /Row 2 -> /Row 3
- D25 pad 1: /Row 2 -> /Row 0
- D26 pad 1: /Row 2 -> /Row 1
- D28 pad 1: /Row 2 -> /Row 3
- D29 pad 1: /Row 2 -> /Row 0
- D30 pad 1: /Row 2 -> /Row 1
- D31 pad 1: /Row 3 -> /Row 2
- D33 pad 1: /Row 3 -> /Row 0
- D34 pad 1: /Row 3 -> /Row 1
- D35 pad 1: /Row 3 -> /Row 2
- D37 pad 1: /Row 3 -> /Row 0
- D38 pad 1: /Row 3 -> /Row 1
- D39 pad 1: /Row 3 -> /Row 2
- D6 pad 1: /Row 0 -> /Row 1
- D7 pad 1: /Row 0 -> /Row 1
- D8 pad 1: /Row 0 -> /Row 1
- D9 pad 1: /Row 0 -> /Row 1
- MX10 pad 1: Net-(MX10-Pad1) -> /Col 6
- MX10 pad 2: Net-(D10-A) -> Net-(D25-A)
- MX11 pad 2: Net-(D11-A) -> Net-(D6-A)
- MX12 pad 2: Net-(D12-A) -> Net-(D7-A)
- MX13 pad 2: Net-(D13-A) -> Net-(D8-A)
- MX14 pad 2: Net-(D14-A) -> Net-(D9-A)
- MX15 pad 2: Net-(D15-A) -> Net-(D10-A)
- MX16 pad 1: /Col 5 -> /Col 0
- MX16 pad 2: Net-(D16-A) -> Net-(D11-A)
- MX17 pad 1: /Col 6 -> /Col 1
- MX17 pad 2: Net-(D17-A) -> Net-(D12-A)
- MX18 pad 1: Net-(MX18-Pad1) -> /Col 2
- MX18 pad 2: Net-(D18-A) -> Net-(D13-A)
- MX19 pad 1: Net-(MX19-Pad1) -> /Col 3
- MX19 pad 2: Net-(D19-A) -> Net-(D14-A)
- MX20 pad 1: Net-(MX10-Pad1) -> /Col 4
- MX20 pad 2: Net-(D20-A) -> Net-(D15-A)
- MX21 pad 2: Net-(D21-A) -> Net-(D16-A)
- MX22 pad 2: Net-(D22-A) -> Net-(D17-A)
- MX23 pad 2: Net-(D23-A) -> Net-(D18-A)
- MX24 pad 2: Net-(D24-A) -> Net-(D19-A)
- MX25 pad 2: Net-(D25-A) -> Net-(D20-A)
- MX26 pad 1: /Col 5 -> /Col 6
- MX28 pad 1: Net-(MX18-Pad1) -> /Col 6
- MX29 pad 1: Net-(MX19-Pad1) -> /Col 7
- MX30 pad 1: Net-(MX10-Pad1) -> /Col 7
- MX31 pad 1: /Col 0 -> /Col 7
- MX32 pad 1: /Col 1 -> /Col 7
- MX33 pad 1: /Col 2 -> /Col 8
- MX34 pad 1: /Col 3 -> /Col 8
- MX35 pad 1: /Col 4 -> /Col 8
- MX36 pad 1: /Col 5 -> /Col 8
- MX37 pad 1: /Col 6 -> /Col 9
- MX38 pad 1: Net-(MX18-Pad1) -> /Col 9
- MX39 pad 1: Net-(MX19-Pad1) -> /Col 9
- MX40 pad 1: Net-(MX10-Pad1) -> /Col 9
- MX6 pad 2: Net-(D6-A) -> Net-(D21-A)
- MX7 pad 1: /Col 6 -> /Col 5
- MX7 pad 2: Net-(D7-A) -> Net-(D22-A)
- MX8 pad 1: Net-(MX18-Pad1) -> /Col 5
- MX8 pad 2: Net-(D8-A) -> Net-(D23-A)
- MX9 pad 1: Net-(MX19-Pad1) -> /Col 5
- MX9 pad 2: Net-(D9-A) -> Net-(D24-A)
Routing:
- net Net-(D8-A): track 7.54 -> 0.00 mm
- net Net-(D7-A): track 7.54 -> 0.00 mm
- net Net-(D1-A): track 7.54 -> 0.00 mm
- net Net-(D4-A): track 7.54 -> 0.00 mm
- net Net-(D3-A): track 7.54 -> 0.00 mm
- net Net-(D2-A): track 7.54 -> 0.00 mm
- net Net-(D9-A): track 7.54 -> 0.00 mm
- net Net-(D6-A): track 7.54 -> 0.00 mm
- net Net-(D10-A): track 7.54 -> 0.00 mm
- net Net-(D17-A): track 7.51 -> 0.00 mm
- net Net-(D27-A): track 7.51 -> 0.00 mm
- net Net-(D11-A): track 7.51 -> 0.00 mm
- net Net-(D31-A): track 7.51 -> 0.00 mm
- net Net-(D21-A): track 7.51 -> 0.00 mm
- net Net-(D14-A): track 7.51 -> 0.00 mm
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Other:
- board size 228.6 x 81 mm -> 261.9 x 76.2 mm
- board text added: "arduino nano goes here :)"
- board text removed: "${REFERENCE}"

Commit message: all wired up
Parts:
- moved D10 275.6 mm to (262.9, 38.1)
- moved D9 257.4 mm to (243.8, 38.1)
- moved D20 255.3 mm to (262.9, 57.1)
- moved D8 239.4 mm to (224.8, 38.1)
- moved D19 236.8 mm to (243.8, 57.1)
- moved D30 236.0 mm to (262.9, 76.2)
- moved D7 221.6 mm to (205.7, 38.1)
- moved D18 218.4 mm to (224.8, 57.1)
- moved D40 217.8 mm to (262.9, 95.2)
- moved D29 217.1 mm to (243.8, 76.2)
- moved D6 204.2 mm to (186.7, 38.1)
- moved D17 200.2 mm to (205.7, 57.1)
- moved D39 198.7 mm to (243.8, 95.2)
- moved D28 198.4 mm to (224.8, 76.2)
- moved D16 182.3 mm to (186.7, 57.1)
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Connections:
- A1 pad 10: unconnected-(A1-D7-Pad10) -> /Col 8
- A1 pad 11: unconnected-(A1-D8-Pad11) -> /Col 7
- A1 pad 12: unconnected-(A1-D9-Pad12) -> /Col 6
- A1 pad 13: unconnected-(A1-D10-Pad13) -> /Col 5
- A1 pad 19: unconnected-(A1-A0-Pad19) -> /Col 4
- A1 pad 20: unconnected-(A1-A1-Pad20) -> /Col 3
- A1 pad 21: unconnected-(A1-A2-Pad21) -> /Col 2
- A1 pad 25: unconnected-(A1-A6-Pad25) -> /Col 1
- A1 pad 26: unconnected-(A1-A7-Pad26) -> /Col 0
- A1 pad 5: unconnected-(A1-D2-Pad5) -> /Row 3
- A1 pad 6: unconnected-(A1-D3-Pad6) -> /Row 2
- A1 pad 7: unconnected-(A1-D4-Pad7) -> /Row 1
- A1 pad 8: unconnected-(A1-D5-Pad8) -> /Row 0
- A1 pad 9: unconnected-(A1-D6-Pad9) -> /Col 9
- D10 pad 1: /Row 1 -> /Row 0
- D11 pad 1: /Row 2 -> /Row 1
- D12 pad 1: /Row 2 -> /Row 1
- D13 pad 1: /Row 2 -> /Row 1
- D14 pad 1: /Row 2 -> /Row 1
- D15 pad 1: /Row 2 -> /Row 1
- D16 pad 1: /Row 3 -> /Row 1
- D17 pad 1: /Row 3 -> /Row 1
- D18 pad 1: /Row 3 -> /Row 1
- D19 pad 1: /Row 3 -> /Row 1
- D20 pad 1: /Row 3 -> /Row 1
- D21 pad 1: /Row 0 -> /Row 2
- D22 pad 1: /Row 1 -> /Row 2
- D24 pad 1: /Row 3 -> /Row 2
- D25 pad 1: /Row 0 -> /Row 2
- D26 pad 1: /Row 1 -> /Row 2
- D28 pad 1: /Row 3 -> /Row 2
- D29 pad 1: /Row 0 -> /Row 2
- D30 pad 1: /Row 1 -> /Row 2
- D31 pad 1: /Row 2 -> /Row 3
- D33 pad 1: /Row 0 -> /Row 3
- D34 pad 1: /Row 1 -> /Row 3
- D35 pad 1: /Row 2 -> /Row 3
- D37 pad 1: /Row 0 -> /Row 3
- D38 pad 1: /Row 1 -> /Row 3
- D39 pad 1: /Row 2 -> /Row 3
- D6 pad 1: /Row 1 -> /Row 0
- D7 pad 1: /Row 1 -> /Row 0
- D8 pad 1: /Row 1 -> /Row 0
- D9 pad 1: /Row 1 -> /Row 0
- MX10 pad 1: /Col 6 -> /Col 9
- MX10 pad 2: Net-(D25-A) -> Net-(D10-A)
- MX11 pad 2: Net-(D6-A) -> Net-(D11-A)
- MX12 pad 2: Net-(D7-A) -> Net-(D12-A)
- MX13 pad 2: Net-(D8-A) -> Net-(D13-A)
- MX14 pad 2: Net-(D9-A) -> Net-(D14-A)
- MX15 pad 2: Net-(D10-A) -> Net-(D15-A)
- MX16 pad 1: /Col 0 -> /Col 5
- MX16 pad 2: Net-(D11-A) -> Net-(D16-A)
- MX17 pad 1: /Col 1 -> /Col 6
- MX17 pad 2: Net-(D12-A) -> Net-(D17-A)
- MX18 pad 1: /Col 2 -> /Col 7
- MX18 pad 2: Net-(D13-A) -> Net-(D18-A)
- MX19 pad 1: /Col 3 -> /Col 8
- MX19 pad 2: Net-(D14-A) -> Net-(D19-A)
- MX20 pad 1: /Col 4 -> /Col 9
- MX20 pad 2: Net-(D15-A) -> Net-(D20-A)
- MX21 pad 2: Net-(D16-A) -> Net-(D21-A)
- MX22 pad 2: Net-(D17-A) -> Net-(D22-A)
- MX23 pad 2: Net-(D18-A) -> Net-(D23-A)
- MX24 pad 2: Net-(D19-A) -> Net-(D24-A)
- MX25 pad 2: Net-(D20-A) -> Net-(D25-A)
- MX26 pad 1: /Col 6 -> /Col 5
- MX28 pad 1: /Col 6 -> /Col 7
- MX29 pad 1: /Col 7 -> /Col 8
- MX30 pad 1: /Col 7 -> /Col 9
- MX31 pad 1: /Col 7 -> /Col 0
- MX32 pad 1: /Col 7 -> /Col 1
- MX33 pad 1: /Col 8 -> /Col 2
- MX34 pad 1: /Col 8 -> /Col 3
- MX35 pad 1: /Col 8 -> /Col 4
- MX36 pad 1: /Col 8 -> /Col 5
- MX37 pad 1: /Col 9 -> /Col 6
- MX38 pad 1: /Col 9 -> /Col 7
- MX39 pad 1: /Col 9 -> /Col 8
- MX6 pad 2: Net-(D21-A) -> Net-(D6-A)
- MX7 pad 1: /Col 5 -> /Col 6
- MX7 pad 2: Net-(D22-A) -> Net-(D7-A)
- MX8 pad 1: /Col 5 -> /Col 7
- MX8 pad 2: Net-(D23-A) -> Net-(D8-A)
- MX9 pad 1: /Col 5 -> /Col 8
- MX9 pad 2: Net-(D24-A) -> Net-(D9-A)
Routing:
- net /Row 3: track 0.00 -> 312.3 mm
- net /Row 2: track 0.00 -> 295.9 mm, vias 0 -> 20
- net /Row 1: track 0.00 -> 288.8 mm, vias 0 -> 19
- net /Row 0: track 0.00 -> 248.6 mm, vias 0 -> 19
- net /Col 0: track 0.00 -> 190.0 mm, vias 0 -> 10
- net /Col 9: track 0.00 -> 180.1 mm, vias 0 -> 2
- net /Col 1: track 0.00 -> 170.8 mm, vias 0 -> 8
- net /Col 8: track 0.00 -> 164.6 mm, vias 0 -> 2
- net /Col 2: track 0.00 -> 151.5 mm, vias 0 -> 6
- net /Col 7: track 0.00 -> 144.0 mm, vias 0 -> 2
- net /Col 3: track 0.00 -> 133.9 mm, vias 0 -> 4
- net /Col 6: track 0.00 -> 125.6 mm, vias 0 -> 2
- net /Col 4: track 0.00 -> 113.3 mm, vias 0 -> 2
- net /Col 5: track 0.00 -> 106.5 mm
- net Net-(A1-GND-Pad29): track 0.00 -> 17.3 mm
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Other:
- board size 261.9 x 76.2 mm -> 257.2 x 78.6 mm
- board text added: "arduino nano :)"
- board text removed: "arduino nano goes here :)"
