File: board/milki.kicad_sch (KiCad schematic)
At the start: 82 parts, among them SW1 SW_Push

Commit message: i've switched up
Parts:
- removed A1: RaspberryPi_Pico, Module:RaspberryPi_Pico_Common_Unspecified, symbol MCU_Module:RaspberryPi_Pico
- added A1: Arduino_Nano_Every, Module:Arduino_Nano, symbol MCU_Module:Arduino_Nano_Every
- MX1, MX10, MX11, MX12, MX13, MX14, MX15, MX16, MX17, MX18, MX19, MX2, MX20, MX21, MX22, MX23, MX24, MX25, MX26, MX27, MX28, MX29, MX3, MX30, MX31, MX32, MX33, MX34, MX35, MX36, MX37, MX38, MX39, MX4, MX40, MX5, MX6, MX7, MX8, MX9: footprint PCM_marbastlib-mx:SW_MX_1u -> MX_Solderable:Low Profile GC plus MX
Connections:
- net Col 0: now also MX16.1; no longer MX31.1
- net Col 1: now also MX17.1; no longer MX32.1
- net Col 2: now also MX18.1; no longer MX33.1
- net Col 3: now also MX19.1; no longer MX34.1
- net Col 4: now also MX20.1; no longer MX35.1
- net Col 5: now also MX7.1, MX8.1, MX9.1; no longer MX16.1, MX26.1, MX36.1
- net Col 6: now also MX10.1, MX26.1, MX28.1; no longer MX17.1, MX37.1, MX7.1
- net Col 7: now also MX29.1, MX30.1, MX31.1, MX32.1
- net Col 8: now also MX33.1, MX34.1, MX35.1, MX36.1
- net Col 9: now also MX37.1, MX38.1, MX39.1, MX40.1
- net Row 0: now also D21.1 (K), D25.1 (K), D29.1 (K), D33.1 (K), D37.1 (K); no longer D10.1 (K), D6.1 (K), D7.1 (K), D8.1 (K), D9.1 (K)
- net Row 1: now also D10.1 (K), D22.1 (K), D26.1 (K), D30.1 (K), D34.1 (K), D38.1 (K), D6.1 (K), D7.1 (K), D8.1 (K), D9.1 (K); no longer D11.1 (K), D12.1 (K), D13.1 (K), D14.1 (K), D15.1 (K), D16.1 (K), D17.1 (K), D18.1 (K), D19.1 (K), D20.1 (K)
- net Row 2: now also D11.1 (K), D12.1 (K), D13.1 (K), D14.1 (K), D15.1 (K), D31.1 (K), D35.1 (K), D39.1 (K); no longer D21.1 (K), D22.1 (K), D24.1 (K), D25.1 (K), D26.1 (K), D28.1 (K), D29.1 (K), D30.1 (K)
- net Row 3: now also D16.1 (K), D17.1 (K), D18.1 (K), D19.1 (K), D20.1 (K), D24.1 (K), D28.1 (K); no longer D31.1 (K), D33.1 (K), D34.1 (K), D35.1 (K), D37.1 (K), D38.1 (K), D39.1 (K)
- net at D22.2 (A): now also MX7.2; no longer MX22.2
- net at D8.2 (A): now also MX13.2; no longer MX8.2
- net at D25.2 (A): now also MX10.2; no longer MX25.2
- net at MX23.2: now also D18.2 (A); no longer D23.2 (A)
- net at D7.2 (A): now also MX12.2; no longer MX7.2
- net at MX15.2: now also D10.2 (A); no longer D15.2 (A)
- net at MX19.2: now also D14.2 (A); no longer D19.2 (A)
- net at D16.2 (A): now also MX21.2; no longer MX16.2
- net at MX17.2: now also D12.2 (A); no longer D17.2 (A)
- net at D20.2 (A): now also MX25.2; no longer MX20.2
- net at D24.2 (A): now also MX9.2; no longer MX24.2
- net at D6.2 (A): now also MX11.2; no longer MX6.2
- net at D9.2 (A): now also MX14.2; no longer MX9.2
- net at D21.2 (A): now also MX6.2; no longer MX21.2
- net at D13.2 (A): now also MX18.2; no longer MX13.2
- net at D11.2 (A): now also MX16.2; no longer MX11.2
- new net: A1.29 (GND), A1.4 (GND)
- new net: D17.2 (A), MX22.2
- new net: D19.2 (A), MX24.2
- new net: D23.2 (A), MX8.2
- new net: D15.2 (A), MX20.2
Other:
- moved on the sheet: D1, D2, D3, D4, D5, MX1, MX2, MX3, MX4, MX5

Commit message: all wired up
Parts:
- removed SW1: SW_Push, symbol Switch:SW_Push
Connections:
- net Col 0: now also A1.26 (A7), MX31.1; no longer MX16.1
- net Col 1: now also A1.25 (A6), MX32.1; no longer MX17.1
- net Col 2: now also A1.21 (A2), MX33.1; no longer MX18.1
- net Col 3: now also A1.20 (A1), MX34.1; no longer MX19.1
- net Col 4: now also A1.19 (A0), MX35.1; no longer MX20.1
- net Col 5: now also A1.13 (D10), MX16.1, MX26.1, MX36.1; no longer MX7.1, MX8.1, MX9.1
- net Col 6: now also A1.12 (D9), MX17.1, MX37.1, MX7.1; no longer MX10.1, MX26.1, MX28.1
- net Col 7: now also A1.11 (D8), MX18.1, MX28.1, MX38.1, MX8.1; no longer MX29.1, MX30.1, MX31.1, MX32.1
- net Col 8: now also A1.10 (D7), MX19.1, MX29.1, MX39.1, MX9.1; no longer MX33.1, MX34.1, MX35.1, MX36.1
- net Col 9: now also A1.9 (D6), MX10.1, MX20.1, MX30.1; no longer MX37.1, MX38.1, MX39.1
- net Row 0: now also A1.8 (D5), D10.1 (K), D6.1 (K), D7.1 (K), D8.1 (K), D9.1 (K); no longer D21.1 (K), D25.1 (K), D29.1 (K), D33.1 (K), D37.1 (K)
- net Row 1: now also A1.7 (D4), D11.1 (K), D12.1 (K), D13.1 (K), D14.1 (K), D15.1 (K), D16.1 (K), D17.1 (K), D18.1 (K), D19.1 (K), D20.1 (K); no longer D10.1 (K), D22.1 (K), D26.1 (K), D30.1 (K), D34.1 (K), D38.1 (K), D6.1 (K), D7.1 (K), D8.1 (K), D9.1 (K)
- net Row 2: now also A1.6 (D3), D21.1 (K), D22.1 (K), D24.1 (K), D25.1 (K), D26.1 (K), D28.1 (K), D29.1 (K), D30.1 (K); no longer D11.1 (K), D12.1 (K), D13.1 (K), D14.1 (K), D15.1 (K), D31.1 (K), D35.1 (K), D39.1 (K)
- net Row 3: now also A1.5 (D2), D31.1 (K), D33.1 (K), D34.1 (K), D35.1 (K), D37.1 (K), D38.1 (K), D39.1 (K); no longer D16.1 (K), D17.1 (K), D18.1 (K), D19.1 (K), D20.1 (K), D24.1 (K), D28.1 (K)
- net at MX10.2: now also D10.2 (A); no longer D25.2 (A)
- net at D6.2 (A): now also MX6.2; no longer MX11.2
- net at MX23.2: now also D23.2 (A); no longer D18.2 (A)
- net at D20.2 (A): now also MX20.2; no longer MX25.2
- net at MX19.2: now also D19.2 (A); no longer D14.2 (A)
- net at MX21.2: now also D21.2 (A); no longer D16.2 (A)
- net at MX14.2: now also D14.2 (A); no longer D9.2 (A)
- net at MX16.2: now also D16.2 (A); no longer D11.2 (A)
- net at MX17.2: now also D17.2 (A); no longer D12.2 (A)
- net at D7.2 (A): now also MX7.2; no longer MX12.2
- net at MX15.2: now also D15.2 (A); no longer D10.2 (A)
- net at MX9.2: now also D9.2 (A); no longer D24.2 (A)
- net at D22.2 (A): now also MX22.2; no longer MX7.2
- net at MX24.2: now also D24.2 (A); no longer D19.2 (A)
- net at MX13.2: now also D13.2 (A); no longer D8.2 (A)
- net at MX8.2: now also D8.2 (A); no longer D23.2 (A)
- net at MX18.2: now also D18.2 (A); no longer D13.2 (A)
- new net: D11.2 (A), MX11.2
- new net: D25.2 (A), MX25.2
- new net: D12.2 (A), MX12.2
